File: 24_volt_power_supply/24_volt_power_supply.kicad_pcb (KiCad board)
At the start: 2 copper layers, 75 x 55 mm, 18 parts, among them J1 Conn_01x02_Pin, J2 Conn_01x01_Pin, J3 Conn_01x01_Pin, J4 Screw_Terminal_01x02, J5 Conn_01x01_Pin, J6 Conn_01x01_Pin, K1 Relay_SPDT

Commit message: better placements for inputs and added silkscreens for components
Parts:
- moved J1 6.25 mm to (76.5, 77.8)
- moved J2 6.25 mm to (76.5, 83.2)
Routing:
- net AC: track 75.2 -> 75.9 mm
Changed lines of the file:
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@@
 	(footprint "Connector_Wire:SolderWire-2.5sqmm_1x01_D2.4mm_OD3.6mm"
 		(layer "F.Cu")
-		(at 76.5 77)
+		(at 76.5 83.25)
 		(descr "Soldered wire connection, for a single 2.5 mm² wire, basic insulation, conductor diameter 2.4mm, outer diameter 3.6mm, size source Multi-Contact FLEXI-E 2.5 (https://www.staubli.com/content/dam/ecs/catalogs-brochures/TM/CAB-Main-11014119-en.pdf#page=9), bend radius 3 times outer diameter, generated with kicad-footprint-generator")
 		(tags "connector wire 2.5sqmm")
@@
 		)
 		(property "Value" "1M"
-			(at 3.81 2.37 0)
-			(layer "F.Fab")
+			(at 3.81 0 0)
+			(layer "F.SilkS")
 			(effects
 				(font
@@
 		)
 		(fp_text user "${REFERENCE}"
-			(at 3.81 0 0)
+			(at 3.81 2.55 0)
 			(layer "F.Fab")
 			(effects
@@
 		(property "Value" "100u"
 			(at 1 3.75 0)
-			(layer "F.Fab")
+			(layer "F.SilkS")
 			(effects
 				(font
@@
 	(footprint "Connector_Wire:SolderWire-2.5sqmm_1x02_P7.2mm_D2.4mm_OD3.6mm"
 		(layer "F.Cu")
-		(at 76.5 71.5 90)
+		(at 76.5 77.75 90)
 		(descr "Soldered wire connection, for 2 times 2.5 mm² wires, basic insulation, conductor diameter 2.4mm, outer diameter 3.6mm, size source Multi-Contact FLEXI-E 2.5 (https://www.staubli.com/content/dam/ecs/catalogs-brochures/TM/CAB-Main-11014119-en.pdf#page=9), bend radius 3 times outer diameter, generated with kicad-footprint-generator")
 		(tags "connector wire 2.5sqmm")
@@
 		)
 		(property "Value" "24V"
-			(at 3.81 2.47 0)
-			(layer "F.Fab")
+			(at 3.81 0 0)
+			(layer "F.SilkS")
 			(effects
 				(font
@@
 		)
 		(fp_text user "${REFERENCE}"
-			(at 4.2 0 0)
+			(at 3.81 2.35 0)
 			(layer "F.Fab")
 			(effects
@@
 		)
 		(property "Value" "1u"
-			(at 11.25 7 90)
-			(layer "F.Fab")
+			(at 11.25 0 90)
+			(layer "F.SilkS")
 			(effects
 				(font
@@
 		)
 		(fp_text user "${REFERENCE}"
-			(at 11.25 0 90)
+			(at 11.25 7.05 90)
 			(layer "F.Fab")
 			(effects
@@
 		)
 		(property "Value" "560"
-			(at 10.16 3.62 0)
-			(layer "F.Fab")
+			(at 10.16 0 0)
+			(layer "F.SilkS")
 			(effects
 				(font
@@
 		)
 		(fp_text user "${REFERENCE}"
-			(at 10.16 0 0)
+			(at 10.16 3.55 0)
 			(layer "F.Fab")
 			(effects
@@
 	)
 	(gr_text "AC IN"
-		(at 79.5 68.5 270)
+		(at 79.5 78.5 0)
 		(layer "F.SilkS")
 		(effects
@@
 	)
 	(gr_text "GND"
-		(at 79.5 62 270)
+		(at 79.5 71.5 0)
 		(layer "F.SilkS")
 		(effects
@@
 	)
 	(gr_text "COM"
-		(at 74 82 0)
+		(at 79.5 84 0)
 		(layer "F.SilkS")
 		(effects
@@
 	)
 	(segment
+		(start 81.25 77.75)
+		(end 76.5 77.75)
+		(width 0.5)
+		(layer "F.Cu")
+		(net 3)
+	)
+	(segment
 		(start 121 98.5)
 		(end 123.8825 95.6175)
@@
 	)
 	(segment
-		(start 88.19 74.5)
-		(end 83 74.5)
+		(start 84.5 74.5)
+		(end 81.25 77.75)
 		(width 0.5)
 		(layer "F.Cu")
@@
 	)
 	(segment
-		(start 92.955113 79.265113)
-		(end 88.19 74.5)
-		(width 0.5)
+		(start 76.95 77.3)
+		(end 76.5 77.75)
+		(width 0.2)
 		(layer "F.Cu")
 		(net 3)
 	)
 	(segment
-		(start 83 74.5)
-		(end 80 71.5)
-		(width 0.5)
-		(layer "F.Cu")
-		(net 3)
-	)
-	(segment
-		(start 80 71.5)
-		(end 76.5 71.5)
+		(start 92.955113 79.265113)
+		(end 88.19 74.5)
 		(width 0.5)
 		(layer "F.Cu")
@@
 	)
 	(segment
-		(start 76.5 71.5)
-		(end 76.5 77)
+		(start 76.5 77.75)
+		(end 76.5 83.25)
 		(width 4)
 		(layer "F.Cu")
@@
 	)
 	(segment
+		(start 88.19 74.5)
+		(end 84.5 74.5)
+		(width 0.5)
+		(layer "F.Cu")
+		(net 3)
+	)
+	(segment
 		(start 117.401255 79.981255)
 		(end 120.42 83)
@@
 		(polygon
 			(pts
-				(xy 74 69) (xy 79 69) (xy 79 79.5) (xy 74 79.5)
+				(xy 74 75.25) (xy 79 75.25) (xy 79 85.75) (xy 74 85.75)
 			)
 		)
@@
 				(xy 131.0662 59.414478) (xy 131.264478 59.2162) (xy 131.43931 58.996968) (xy 131.588496 58.759539)
 				(xy 131.710161 58.5069) (xy 131.802774 58.242227) (xy 131.86517 57.968849) (xy 131.896566 57.690204)
-				(xy 131.896566 57.409796)
 			)
 		)
@@
 				(xy 119.13798 59.4329) (xy 119.3329 59.23798) (xy 119.504771 59.022461) (xy 119.65143 58.789054)
 				(xy 119.771034 58.540693) (xy 119.862079 58.280503) (xy 119.923419 58.011755) (xy 119.954283 57.73783)
-				(xy 119.954283 57.46217)
 			)
 		)
@@
 				(xy 125.1162 73.664478) (xy 125.314478 73.4662) (xy 125.48931 73.246968) (xy 125.638496 73.009539)
 				(xy 125.760161 72.7569) (xy 125.852774 72.492227) (xy 125.91517 72.218849) (xy 125.946566 71.940204)
-				(xy 125.946566 71.659796)
 			)
 		)

Commit message: better placements for inputs and added silkscreens for components
Other:
- board text added: "24V TO SWITCH"
Changed lines of the file:
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@@
 		)
 		(property "Value" "Screw_Terminal_01x02"
-			(at 1.5 5.5 0)
+			(at 2.5 -9.1175 0)
 			(layer "F.Fab")
 			(effects
@@
 		(layer "F.SilkS")
 		(effects
+			(font
+				(size 1.5 1.5)
+				(thickness 0.3)
+				(bold yes)
+			)
+			(justify left bottom)
+		)
+	)
+	(gr_text "24V TO SWITCH"
+		(at 118 103 0)
+		(layer "F.SilkS")
+		(effects

Commit message: added location for product No (PCBWay)
Other:
- board text added: "WayWayWay"
Changed lines of the file:
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@@
+		)
+	)
+	(gr_text "WayWayWay"
+		(at 145 82.5 90)
+		(layer "F.SilkS")
+		(effects
+			(font
+				(size 1 1)
+				(thickness 0.1)
+			)
+			(justify left bottom)
 		)
 	)

Commit message: added warning lables
Parts:
- added G***: LOGO, test:high_voltage_image, F.Cu at (136.5, 94.5)
Other:
- board text added: "Warning! Unisolated Mains Voltage! Do Not Touch Or Work On Board When On!"
Changed lines of the file:
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@@
 	(net 8 "Net-(J6-Pin_1)")
 	(net 9 "Net-(J5-Pin_1)")
+	(footprint "test:high_voltage_image"
+		(layer "F.Cu")
+		(at 136.5 94.5 90)
+		(property "Reference" "G***"
+			(at 0 0 90)
+			(layer "F.SilkS")
+			(hide yes)
+			(effects
+				(font
+					(size 1.5 1.5)
+					(thickness 0.3)
+				)
+			)
+		)
+		(property "Value" "LOGO"
+			(at 0.75 0 90)
+			(layer "F.SilkS")
+			(hide yes)
+			(effects
+				(font
+					(size 1.5 1.5)
+					(thickness 0.3)
+				)
+			)
+		)
+		(property "Datasheet" ""
+			(at 0 0 90)
+			(layer "F.Fab")
+			(hide yes)
+			(effects
+				(font
+					(size 1.27 1.27)
+					(thickness 0.15)
+				)
+			)
+		)
+		(property "Description" ""
+			(at 0 0 90)
+			(layer "F.Fab")
+			(hide yes)
+			(effects
+				(font
+					(size 1.27 1.27)
+					(thickness 0.15)
+				)
+			)
+		)
+		(attr board_only exclude_from_pos_files exclude_from_bom)
+		(fp_poly
+			(pts
+				(xy 0.320036 -0.907389) (xy 0.389272 -0.902694) (xy 0.424069 -0.893947) (xy 0.430177 -0.880394)
+				(xy 0.430029 -0.880028) (xy 0.417996 -0.852394) (xy 0.389777 -0.788134) (xy 0.34778 -0.692716) (xy 0.294413 -0.571603)
+				(xy 0.232082 -0.430262) (xy 0.163196 -0.274158) (xy 0.139647 -0.220817) (xy 0.070032 -0.062493)
+				(xy 0.00719 0.081674) (xy -0.046651 0.206478) (xy -0.089266 0.30671) (xy -0.11843 0.377164) (xy -0.131916 0.412633)
+				(xy -0.132511 0.415828) (xy -0.110332 0.409511) (xy -0.052434 0.388199) (xy 0.034398 0.354522) (xy 0.143378 0.31111)
+				(xy 0.263426 0.262354) (xy 0.388117 0.211923) (xy 0.497994 0.16872) (xy 0.586065 0.135395) (xy 0.645338 0.114595)
+				(xy 0.668634 0.108861) (xy 0.666489 0.131682) (xy 0.653345 0.19368) (xy 0.630489 0.289684) (xy 0.59921 0.414529)
+				(xy 0.560794 0.563046) (xy 0.516532 0.730066) (xy 0.480707 0.862771) (xy 0.432317 1.041388) (xy 0.388009 1.206327)
+				(xy 0.349194 1.352217) (xy 0.317288 1.473691) (xy 0.293703 1.565377) (xy 0.279852 1.621907) (xy 0.276701 1.637808)
+				(xy 0.296281 1.659028) (xy 0.34434 1.672202) (xy 0.34543 1.672319) (xy 0.414773 1.679528) (xy 0.23901 1.944111)
+				(xy 0.161391 2.060705) (xy 0.105308 2.143625) (xy 0.066891 2.197563) (xy 0.042269 2.227209) (xy 0.027572 2.237256)
+				(xy 0.018931 2.232395) (xy 0.012825 2.218294) (xy -0.033295 2.089171) (xy -0.077529 1.964444) (xy -0.117277 1.851539)
+				(xy -0.149939 1.75788) (xy -0.172917 1.690892) (xy -0.183609 1.658) (xy -0.184059 1.655998) (xy -0.163777 1.64894)
+				(xy -0.113651 1.641913) (xy -0.100119 1.640654) (xy -0.016179 1.633514) (xy 0.105709 1.20788) (xy 0.14455 1.071969)
+				(xy 0.179636 0.94867) (xy 0.208749 0.845827) (xy 0.229667 0.771282) (xy 0.240171 0.73288) (xy 0.240305 0.732357)
+				(xy 0.241439 0.716149) (xy 0.231013 0.708759) (xy 0.20365 0.711721) (xy 0.153971 0.726568) (xy 0.076599 0.754833)
+				(xy -0.033842 0.798051) (xy -0.142142 0.841412) (xy -0.267357 0.891098) (xy -0.377253 0.933414)
+				(xy -0.465001 0.965836) (xy -0.523775 0.98584) (xy -0.546723 0.990928) (xy -0.542739 0.967472) (xy -0.527376 0.904569)
+				(xy -0.501925 0.807008) (xy -0.467677 0.679577) (xy -0.425922 0.527066) (xy -0.377951 0.354264)
+				(xy -0.325057 0.165959) (xy -0.309546 0.111131) (xy -0.254281 -0.083935) (xy -0.202263 -0.267566)
+				(xy -0.154986 -0.434479) (xy -0.113948 -0.579391) (xy -0.080644 -0.697021) (xy -0.05657 -0.782085)
+				(xy -0.043222 -0.829301) (xy -0.041894 -0.834014) (xy -0.020845 -0.908787) (xy 0.210608 -0.908787)
+			)
+			(stroke
+				(width 0)
+				(type solid)
+			)
+			(fill yes)
+			(layer "F.SilkS")
+		)
+		(fp_poly
+			(pts
+				(xy 0.084597 -2.971744) (xy 0.098459 -2.959187) (xy 0.121024 -2.930611) (xy 0.153269 -2.88438) (xy 0.196171 -2.818859)
+				(xy 0.250708 -2.732413) (xy 0.317857 -2.623407) (xy 0.398594 -2.490205) (xy 0.493899 -2.331174)
+				(xy 0.604746 -2.144676) (xy 0.732115 -1.929078) (xy 0.876982 -1.682744) (xy 1.040324 -1.404039)
+				(xy 1.223118 -1.091328) (xy 1.426343 -0.742976) (xy 1.650974 -0.357347) (xy 1.79397 -0.111634) (xy 2.024226 0.284552)
+				(xy 2.24009 0.656816) (xy 2.440801 1.00382) (xy 2.625597 1.324228) (xy 2.793716 1.616701) (xy 2.944394 1.879903)
+				(xy 3.076871 2.112496) (xy 3.190383 2.313143) (xy 3.284169 2.480506) (xy 3.357466 2.613249) (xy 3.409513 2.710034)
+				(xy 3.439546 2.769523) (xy 3.447179 2.788959) (xy 3.444751 2.848426) (xy 3.415422 2.901051) (xy 3.386273 2.932754)
+				(xy 3.316583 3.002445) (xy -0.000001 3.002445) (xy -3.316584 3.002445) (xy -3.383836 2.935193) (xy -3.437298 2.859293)
+				(xy -3.448134 2.777008) (xy -3.417125 2.681353) (xy -3.413136 2.673449) (xy -3.393437 2.637779)
+				(xy -3.352611 2.565978) (xy -3.292268 2.460809) (xy -3.28951 2.456023) (xy -2.753828 2.456023) (xy -2.732554 2.458227)
+				(xy -2.668068 2.460349) (xy -2.563173 2.462373) (xy -2.42067 2.464279) (xy -2.243363 2.466051) (xy -2.034054 2.46767)
+				(xy -1.795546 2.46912) (xy -1.53064 2.470383) (xy -1.24214 2.47144) (xy -0.932848 2.472275) (xy -0.605566 2.472869)
+				(xy -0.263097 2.473206) (xy -0.0104 2.473278) (xy 0.40841 2.473221) (xy 0.783503 2.473033) (xy 1.117174 2.472685)
+				(xy 1.411719 2.47215) (xy 1.669436 2.471401) (xy 1.892621 2.47041) (xy 2.08357 2.46915) (xy 2.244578 2.467594)
+				(xy 2.377944 2.465713) (xy 2.485963 2.463481) (xy 2.570931 2.46087) (xy 2.635146 2.457852) (xy 2.680903 2.4544)
+				(xy 2.710498 2.450487) (xy 2.726229 2.446085) (xy 2.730391 2.441166) (xy 2.730208 2.440503) (xy 2.717814 2.417808)
+				(xy 2.684277 2.358224) (xy 2.631333 2.264788) (xy 2.560715 2.140534) (xy 2.474162 1.988497) (xy 2.373407 1.811714)
+				(xy 2.260187 1.613218) (xy 2.136237 1.396046) (xy 2.003294 1.163232) (xy 1.863092 0.917812) (xy 1.717367 0.662821)
+				(xy 1.567855 0.401295) (xy 1.416292 0.136268) (xy 1.264413 -0.129225) (xy 1.113954 -0.392147) (xy 0.96665 -0.649464)
+				(xy 0.824238 -0.89814) (xy 0.688452 -1.135141) (xy 0.561029 -1.357431) (xy 0.443704 -1.561975) (xy 0.338212 -1.745737)
+				(xy 0.24629 -1.905683) (xy 0.169673 -2.038776) (xy 0.110097 -2.141983) (xy 0.08724 -2.181432) (xy -0.003776 -2.338225)
+				(xy -0.11987 -2.135417) (xy -0.146963 -2.088134) (xy -0.195305 -2.003817) (xy -0.263246 -1.885346)
+				(xy -0.349133 -1.735599) (xy -0.451317 -1.557453) (xy -0.568146 -1.353787) (xy -0.697968 -1.12748)
+				(xy -0.839133 -0.88141) (xy -0.98999 -0.618454) (xy -1.148888 -0.341492) (xy -1.314174 -0.053401)
+				(xy -1.484199 0.24294) (xy -1.490017 0.253079) (xy -1.657626 0.545207) (xy -1.818836 0.826186) (xy -1.972166 1.093436)
+				(xy -2.116138 1.344378) (xy -2.24927 1.576431) (xy -2.370083 1.787017) (xy -2.477097 1.973554) (xy -2.568831 2.133464)
+				(xy -2.643806 2.264166) (xy -2.700542 2.363082) (xy -2.737559 2.427629) (xy -2.753376 2.455231)
+				(xy -2.753828 2.456023) (xy -3.28951 2.456023) (xy -3.214018 2.325036) (xy -3.119471 2.16142) (xy -3.010234 1.972726)
+				(xy -2.887919 1.761716) (xy -2.754135 1.531152) (xy -2.61049 1.283798) (xy -2.458596 1.022417) (xy -2.30006 0.74977)
+				(xy -2.136493 0.468622) (xy -1.969505 0.181736) (xy -1.800704 -0.108127) (xy -1.6317 -0.398203)
+				(xy -1.464103 -0.685729) (xy -1.299522 -0.967943) (xy -1.139567 -1.242081) (xy -0.985847 -1.505381)
+				(xy -0.839972 -1.75508) (xy -0.703551 -1.988414) (xy -0.578194 -2.202622) (xy -0.46551 -2.39494)
+				(xy -0.367109 -2.562605) (xy -0.2846 -2.702854) (xy -0.219592 -2.812925) (xy -0.173697 -2.890055)
+				(xy -0.148521 -2.931481) (xy -0.144269 -2.937873) (xy -0.078614 -2.981202) (xy 0.00452 -2.993031)
+			)
+			(stroke
+				(width 0)
+				(type solid)
+			)
+			(fill yes)
+			(layer "F.SilkS")
+		)
+		(embedded_fonts no)
+	)
 	(footprint "MountingHole:MountingHole_3.2mm_M3_ISO14580_Pad_TopOnly"
 		(layer "F.Cu")
@@
 		)
 	)
+	(gr_text "Warning! Unisolated Mains Voltage!\nDo Not Touch Or Work On Board When On!"
+		(at 142.5 76.5 90)
+		(layer "F.SilkS")
+		(effects
+			(font
+				(size 1 1)
+				(thickness 0.25)
+				(bold yes)
+			)
+			(justify bottom)
+		)
+	)
